Commit message: Add loader linkage kinematics tools

File: ros_ws/src/loader_description/urdf/loader.urdf.xacro (robot description, xacro)
@@ -118,5 +118,5 @@
     <parent link="front_frame"/><child link="lift_arm"/>
     <origin xyz="0.75 0 0.65" rpy="0 0 0"/>
-    <axis xyz="0 1 0"/>
+    <axis xyz="0 -1 0"/>
     <limit lower="-0.20" upper="1.10" effort="600000" velocity="0.45"/>
     <dynamics damping="30000" friction="5000"/>
@@ -128,5 +128,5 @@
     <parent link="lift_arm"/><child link="bucket"/>
     <origin xyz="2.8 0 0" rpy="0 0 0"/>
-    <axis xyz="0 1 0"/>
+    <axis xyz="0 -1 0"/>
     <limit lower="-1.20" upper="0.80" effort="500000" velocity="0.55"/>
     <dynamics damping="25000" friction="4000"/>

Commit message: 9/4早上的进展

File: ros_ws/src/loader_description/urdf/loader.urdf.xacro (robot description, xacro)
@@ -7,4 +7,7 @@
   -->
   <xacro:arg name="model_fidelity" default="nominal"/>
+  <xacro:arg name="enable_dynamics" default="false"/>
+  <xacro:arg name="enable_lidar_imu" default="false"/>
+  <xacro:arg name="enable_ros2_control" default="false"/>
   <xacro:property name="nominal_track" value="2.5"/>
   <xacro:property name="nominal_wheel_radius" value="0.75"/>
@@ -132,13 +135,126 @@
     <dynamics damping="25000" friction="4000"/>
   </joint>
-  <link name="lidar_link"/>
+  <link name="lidar_link">
+    <inertial>
+      <mass value="2.0"/>
+      <inertia ixx="0.008" ixy="0" ixz="0" iyy="0.008" iyz="0" izz="0.008"/>
+    </inertial>
+  </link>
   <joint name="lidar_mount_joint" type="fixed">
     <parent link="rear_frame"/><child link="lidar_link"/>
     <origin xyz="-0.85 0 2.25" rpy="0 0 0"/>
   </joint>
-  <link name="imu_link"/>
+  <gazebo reference="lidar_mount_joint">
+    <preserveFixedJoint>true</preserveFixedJoint>
+  </gazebo>
+  <link name="imu_link">
+    <inertial>
+      <mass value="0.2"/>
+      <inertia ixx="0.0002" ixy="0" ixz="0" iyy="0.0002" iyz="0" izz="0.0002"/>
+    </inertial>
+  </link>
   <joint name="imu_mount_joint" type="fixed">
     <parent link="rear_frame"/><child link="imu_link"/>
     <origin xyz="-0.2 0 0.65" rpy="0 0 0"/>
   </joint>
+  <gazebo reference="imu_mount_joint">
+    <preserveFixedJoint>true</preserveFixedJoint>
+  </gazebo>
+  <xacro:if value="$(arg enable_ros2_control)">
+    <ros2_control name="LoaderGazeboSystem" type="system">
+      <hardware>
+        <plugin>gz_ros2_control/GazeboSimSystem</plugin>
+      </hardware>
+      <joint name="front_left_wheel_joint">
+        <command_interface name="effort"><param name="min">-20000</param><param name="max">20000</param></command_interface>
+        <state_interface name="position"/><state_interface name="velocity"/>
+      </joint>
+      <joint name="front_right_wheel_joint">
+        <command_interface name="effort"><param name="min">-20000</param><param name="max">20000</param></command_interface>
+        <state_interface name="position"/><state_interface name="velocity"/>
+      </joint>
+      <joint name="rear_left_wheel_joint">
+        <command_interface name="effort"><param name="min">-20000</param><param name="max">20000</param></command_interface>
+        <state_interface name="position"/><state_interface name="velocity"/>
+      </joint>
+      <joint name="rear_right_wheel_joint">
+        <command_interface name="effort"><param name="min">-20000</param><param name="max">20000</param></command_interface>
+        <state_interface name="position"/><state_interface name="velocity"/>
+      </joint>
+      <joint name="articulation_joint">
+        <command_interface name="effort"><param name="min">-250000</param><param name="max">250000</param></command_interface>
+        <state_interface name="position"/><state_interface name="velocity"/>
+      </joint>
+      <joint name="rear_axle_oscillation_joint">
+        <state_interface name="position"/><state_interface name="velocity"/>
+      </joint>
+      <joint name="lift_joint">
+        <command_interface name="effort"><param name="min">-600000</param><param name="max">600000</param></command_interface>
+        <state_interface name="position"/><state_interface name="velocity"/>
+      </joint>
+      <joint name="bucket_tilt_joint">
+        <command_interface name="effort"><param name="min">-500000</param><param name="max">500000</param></command_interface>
+        <state_interface name="position"/><state_interface name="velocity"/>
+      </joint>
+    </ros2_control>
+    <gazebo>
+      <plugin filename="gz_ros2_control-system" name="gz_ros2_control::GazeboSimROS2ControlPlugin">
+        <parameters>$(find loader_control)/config/loader_controllers.yaml</parameters>
+      </plugin>
+    </gazebo>
+  </xacro:if>
+  <xacro:if value="$(arg enable_lidar_imu)">
+    <gazebo reference="lidar_link">
+      <sensor name="loader_gpu_lidar" type="gpu_lidar">
+        <always_on>true</always_on>
+        <update_rate>10</update_rate>
+        <visualize>false</visualize>
+        <topic>/loader/sensors/lidar/scan</topic>
+        <lidar>
+          <scan>
+            <horizontal>
+              <samples>1024</samples>
+              <resolution>1</resolution>
+              <min_angle>${-pi}</min_angle>
+              <max_angle>${pi}</max_angle>
+            </horizontal>
+            <vertical>
+              <samples>32</samples>
+              <resolution>1</resolution>
+              <min_angle>-0.436332</min_angle>
+              <max_angle>0.261799</max_angle>
+            </vertical>
+          </scan>
+          <range>
+            <min>0.5</min>
+            <max>120.0</max>
+            <resolution>0.02</resolution>
+          </range>
+          <noise>
+            <type>gaussian</type>
+            <mean>0.0</mean>
+            <stddev>0.02</stddev>
+          </noise>
+        </lidar>
+      </sensor>
+    </gazebo>
+    <gazebo reference="imu_link">
+      <sensor name="loader_imu" type="imu">
+        <always_on>true</always_on>
+        <update_rate>100</update_rate>
+        <visualize>false</visualize>
+        <topic>/loader/sensors/imu</topic>
+      </sensor>
+    </gazebo>
+  </xacro:if>
+  <xacro:if value="$(arg enable_dynamics)">
+    <gazebo>
+      <plugin filename="libloader_dynamics_system.so" name="loader_sim::LoaderDynamicsSystem">
+        <command_topic>/loader/command</command_topic>
+        <state_topic>/loader/state</state_topic>
+        <command_timeout_s>0.5</command_timeout_s>
+        <state_rate_hz>50</state_rate_hz>
+      </plugin>
+    </gazebo>
+  </xacro:if>
 </robot>

Commit message: chore: sync updates 2026-09-04 21:00 CST

File: ros_ws/src/loader_description/urdf/loader.urdf.xacro (robot description, xacro)
@@ -10,4 +10,5 @@
   <xacro:arg name="enable_lidar_imu" default="false"/>
   <xacro:arg name="enable_ros2_control" default="false"/>
+  <xacro:arg name="enable_soil_slice" default="false"/>
   <xacro:property name="nominal_track" value="2.5"/>
   <xacro:property name="nominal_wheel_radius" value="0.75"/>
@@ -258,3 +259,29 @@
     </gazebo>
   </xacro:if>
+  <xacro:if value="$(arg enable_soil_slice)">
+    <gazebo reference="bucket">
+      <collision name="bucket_collision">
+        <surface>
+          <contact><collide_bitmask>0x01</collide_bitmask></contact>
+        </surface>
+      </collision>
+    </gazebo>
+    <gazebo>
+      <plugin filename="libloader_soil_slice_system.so" name="loader_soil::LoaderSoilSliceSystem">
+        <domain_min_m>0.0</domain_min_m>
+        <domain_max_m>14.0</domain_max_m>
+        <cell_size_m>0.05</cell_size_m>
+        <slice_width_m>2.7</slice_width_m>
+        <pile_center_m>7.0</pile_center_m>
+        <pile_height_m>1.8</pile_height_m>
+        <angle_of_repose_deg>34.0</angle_of_repose_deg>
+        <bucket_capacity_m3>3.0</bucket_capacity_m3>
+        <bulk_density_kg_m3>1600.0</bulk_density_kg_m3>
+        <visualization_update_hz>10.0</visualization_update_hz>
+        <visualization_column_height_m>1.8</visualization_column_height_m>
+        <unload_tilt_threshold_rad>-0.35</unload_tilt_threshold_rad>
+        <maximum_unload_rate_m3ps>3.0</maximum_unload_rate_m3ps>
+      </plugin>
+    </gazebo>
+  </xacro:if>
 </robot>

Commit message: 第四阶段 M1：IMU 名义噪声模型、雷达效应通道与传感器安装扰动

File: ros_ws/src/loader_description/urdf/loader.urdf.xacro (robot description, xacro)
@@ -11,4 +11,18 @@
   <xacro:arg name="enable_ros2_control" default="false"/>
   <xacro:arg name="enable_soil_slice" default="false"/>
+  <!-- Nominal mid-grade MEMS IMU errors; replace with the target unit's datasheet. -->
+  <xacro:arg name="imu_gyro_noise_stddev" default="0.0017"/>
+  <xacro:arg name="imu_gyro_bias_stddev" default="0.00017"/>
+  <xacro:arg name="imu_accel_noise_stddev" default="0.017"/>
+  <xacro:arg name="imu_accel_bias_stddev" default="0.0017"/>
+  <!-- Calibration perturbations added to the nominal sensor mounts. -->
+  <xacro:arg name="lidar_mount_offset_xyz" default="0 0 0"/>
+  <xacro:arg name="lidar_mount_offset_rpy" default="0 0 0"/>
+  <xacro:arg name="imu_mount_offset_xyz" default="0 0 0"/>
+  <xacro:arg name="imu_mount_offset_rpy" default="0 0 0"/>
+  <xacro:property name="lidar_off_xyz" value="${[float(v) for v in '$(arg lidar_mount_offset_xyz)'.split()]}"/>
+  <xacro:property name="lidar_off_rpy" value="${[float(v) for v in '$(arg lidar_mount_offset_rpy)'.split()]}"/>
+  <xacro:property name="imu_off_xyz" value="${[float(v) for v in '$(arg imu_mount_offset_xyz)'.split()]}"/>
+  <xacro:property name="imu_off_rpy" value="${[float(v) for v in '$(arg imu_mount_offset_rpy)'.split()]}"/>
   <xacro:property name="nominal_track" value="2.5"/>
   <xacro:property name="nominal_wheel_radius" value="0.75"/>
@@ -144,5 +158,6 @@
   <joint name="lidar_mount_joint" type="fixed">
     <parent link="rear_frame"/><child link="lidar_link"/>
-    <origin xyz="-0.85 0 2.25" rpy="0 0 0"/>
+    <origin xyz="${-0.85 + lidar_off_xyz[0]} ${lidar_off_xyz[1]} ${2.25 + lidar_off_xyz[2]}"
+      rpy="${lidar_off_rpy[0]} ${lidar_off_rpy[1]} ${lidar_off_rpy[2]}"/>
   </joint>
   <gazebo reference="lidar_mount_joint">
@@ -157,5 +172,6 @@
   <joint name="imu_mount_joint" type="fixed">
     <parent link="rear_frame"/><child link="imu_link"/>
-    <origin xyz="-0.2 0 0.65" rpy="0 0 0"/>
+    <origin xyz="${-0.2 + imu_off_xyz[0]} ${imu_off_xyz[1]} ${0.65 + imu_off_xyz[2]}"
+      rpy="${imu_off_rpy[0]} ${imu_off_rpy[1]} ${imu_off_rpy[2]}"/>
   </joint>
   <gazebo reference="imu_mount_joint">
@@ -246,4 +262,16 @@
         <visualize>false</visualize>
         <topic>/loader/sensors/imu</topic>
+        <imu>
+          <angular_velocity>
+            <x><noise type="gaussian"><mean>0</mean><stddev>$(arg imu_gyro_noise_stddev)</stddev><bias_mean>0</bias_mean><bias_stddev>$(arg imu_gyro_bias_stddev)</bias_stddev></noise></x>
+            <y><noise type="gaussian"><mean>0</mean><stddev>$(arg imu_gyro_noise_stddev)</stddev><bias_mean>0</bias_mean><bias_stddev>$(arg imu_gyro_bias_stddev)</bias_stddev></noise></y>
+            <z><noise type="gaussian"><mean>0</mean><stddev>$(arg imu_gyro_noise_stddev)</stddev><bias_mean>0</bias_mean><bias_stddev>$(arg imu_gyro_bias_stddev)</bias_stddev></noise></z>
+          </angular_velocity>
+          <linear_acceleration>
+            <x><noise type="gaussian"><mean>0</mean><stddev>$(arg imu_accel_noise_stddev)</stddev><bias_mean>0</bias_mean><bias_stddev>$(arg imu_accel_bias_stddev)</bias_stddev></noise></x>
+            <y><noise type="gaussian"><mean>0</mean><stddev>$(arg imu_accel_noise_stddev)</stddev><bias_mean>0</bias_mean><bias_stddev>$(arg imu_accel_bias_stddev)</bias_stddev></noise></y>
+            <z><noise type="gaussian"><mean>0</mean><stddev>$(arg imu_accel_noise_stddev)</stddev><bias_mean>0</bias_mean><bias_stddev>$(arg imu_accel_bias_stddev)</bias_stddev></noise></z>
+          </linear_acceleration>
+        </imu>
       </sensor>
     </gazebo>

Commit message: Add beginner docs and L580 mesh assets

File: ros_ws/src/loader_description/urdf/loader.urdf.xacro (robot description, xacro)
@@ -7,4 +7,7 @@
   -->
   <xacro:arg name="model_fidelity" default="nominal"/>
+  <!-- Visual-only: replace primitive visuals with the L580 wheel-loader meshes.
+       Collisions, inertia, and joints are unchanged, so dynamics are unaffected. -->
+  <xacro:arg name="mesh_visuals" default="true"/>
   <xacro:arg name="enable_dynamics" default="false"/>
   <xacro:arg name="enable_lidar_imu" default="false"/>
@@ -29,8 +32,9 @@
   <xacro:property name="nominal_wheel_radius" value="0.75"/>
   <xacro:property name="nominal_wheel_width" value="0.55"/>
+  <xacro:property name="loader_mesh_dir" value="file:///$(find loader_description)/meshes/l580"/>
   <material name="loader_yellow"><color rgba="0.95 0.58 0.03 1"/></material>
   <material name="loader_dark"><color rgba="0.08 0.09 0.10 1"/></material>
   <material name="bucket_gray"><color rgba="0.28 0.30 0.32 1"/></material>
-  <xacro:macro name="box_link" params="name mass size_x size_y size_z geometry_xyz material">
+  <xacro:macro name="box_link" params="name mass size_x size_y size_z geometry_xyz material mesh:=''">
     <link name="${name}">
       <inertial>
@@ -43,6 +47,13 @@
       </inertial>
       <visual>
-        <origin xyz="${geometry_xyz}" rpy="0 0 0"/>
-        <geometry><box size="${size_x} ${size_y} ${size_z}"/></geometry>
+        <xacro:if value="${mesh != '' and '$(arg mesh_visuals)' == 'true'}">
+          <!-- Mesh is baked into the link frame; keep the primitive as collision. -->
+          <origin xyz="0 0 0" rpy="0 0 0"/>
+          <geometry><mesh filename="${mesh}"/></geometry>
+        </xacro:if>
+        <xacro:unless value="${mesh != '' and '$(arg mesh_visuals)' == 'true'}">
+          <origin xyz="${geometry_xyz}" rpy="0 0 0"/>
+          <geometry><box size="${size_x} ${size_y} ${size_z}"/></geometry>
+        </xacro:unless>
         <material name="${material}"/>
       </visual>
@@ -66,6 +77,13 @@
       </inertial>
       <visual>
-        <origin xyz="0 0 0" rpy="${pi / 2.0} 0 0"/>
-        <geometry><cylinder radius="${nominal_wheel_radius}" length="${nominal_wheel_width}"/></geometry>
+        <xacro:if value="'$(arg mesh_visuals)' == 'true'">
+          <!-- Mesh is centered on the link frame with the axle along +y. -->
+          <origin xyz="0 0 0" rpy="0 0 0"/>
+          <geometry><mesh filename="${loader_mesh_dir}/wheel.STL"/></geometry>
+        </xacro:if>
+        <xacro:unless value="'$(arg mesh_visuals)' == 'true'">
+          <origin xyz="0 0 0" rpy="${pi / 2.0} 0 0"/>
+          <geometry><cylinder radius="${nominal_wheel_radius}" length="${nominal_wheel_width}"/></geometry>
+        </xacro:unless>
         <material name="loader_dark"/>
       </visual>
@@ -79,5 +97,6 @@
   <xacro:box_link
     name="rear_frame" mass="7200" size_x="2.8" size_y="2.2" size_z="0.8"
-    geometry_xyz="-1.4 0 0.15" material="loader_yellow"/>
+    geometry_xyz="-1.4 0 0.15" material="loader_yellow"
+    mesh="${loader_mesh_dir}/rear_body.STL"/>
   <joint name="base_to_rear_frame" type="fixed">
     <parent link="base_link"/>
@@ -87,5 +106,6 @@
   <xacro:box_link
     name="front_frame" mass="6200" size_x="3.0" size_y="2.2" size_z="0.75"
-    geometry_xyz="1.5 0 0.15" material="loader_yellow"/>
+    geometry_xyz="1.5 0 0.15" material="loader_yellow"
+    mesh="${loader_mesh_dir}/front_body.STL"/>
   <joint name="articulation_joint" type="revolute">
     <parent link="rear_frame"/>
@@ -133,5 +153,6 @@
   <xacro:box_link
     name="lift_arm" mass="1200" size_x="2.8" size_y="0.55" size_z="0.35"
-    geometry_xyz="1.4 0 0" material="loader_yellow"/>
+    geometry_xyz="1.4 0 0" material="loader_yellow"
+    mesh="${loader_mesh_dir}/lift_arm.STL"/>
   <joint name="lift_joint" type="revolute">
     <parent link="front_frame"/><child link="lift_arm"/>
@@ -143,5 +164,6 @@
   <xacro:box_link
     name="bucket" mass="1800" size_x="1.25" size_y="2.7" size_z="0.85"
-    geometry_xyz="0.40 0 -0.20" material="bucket_gray"/>
+    geometry_xyz="0.40 0 -0.20" material="bucket_gray"
+    mesh="${loader_mesh_dir}/bucket.STL"/>
   <joint name="bucket_tilt_joint" type="revolute">
     <parent link="lift_arm"/><child link="bucket"/>

Commit message: Refine L580 visual model and localization geometry

File: ros_ws/src/loader_description/urdf/loader.urdf.xacro (robot description, xacro)
@@ -8,5 +8,5 @@
   <xacro:arg name="model_fidelity" default="nominal"/>
   <!-- Visual-only: replace primitive visuals with the L580 wheel-loader meshes.
-       Collisions, inertia, and joints are unchanged, so dynamics are unaffected. -->
+       Collision/inertia remain nominal; rendered geometry affects GPU lidar. -->
   <xacro:arg name="mesh_visuals" default="true"/>
   <xacro:arg name="enable_dynamics" default="false"/>
@@ -36,5 +36,7 @@
   <material name="loader_dark"><color rgba="0.08 0.09 0.10 1"/></material>
   <material name="bucket_gray"><color rgba="0.28 0.30 0.32 1"/></material>
-  <xacro:macro name="box_link" params="name mass size_x size_y size_z geometry_xyz material mesh:=''">
+  <material name="cab_glass"><color rgba="0.035 0.10 0.14 1"/></material>
+  <material name="wheel_rim"><color rgba="0.54 0.57 0.60 1"/></material>
+  <xacro:macro name="box_link" params="name mass size_x size_y size_z geometry_xyz material mesh:='' glass:=false">
     <link name="${name}">
       <inertial>
@@ -58,4 +60,10 @@
         <material name="${material}"/>
       </visual>
+      <xacro:if value="${glass and '$(arg mesh_visuals)' == 'true'}">
+        <visual>
+          <geometry><mesh filename="${loader_mesh_dir}/visual/cab_glass.STL"/></geometry>
+          <material name="cab_glass"/>
+        </visual>
+      </xacro:if>
       <collision>
         <origin xyz="${geometry_xyz}" rpy="0 0 0"/>
@@ -64,5 +72,5 @@
     </link>
   </xacro:macro>
-  <xacro:macro name="wheel_link" params="name mass">
+  <xacro:macro name="wheel_link" params="name mass flip:=0">
     <link name="${name}">
       <inertial>
@@ -77,10 +85,10 @@
       </inertial>
       <visual>
-        <xacro:if value="'$(arg mesh_visuals)' == 'true'">
+        <xacro:if value="$(arg mesh_visuals)">
           <!-- Mesh is centered on the link frame with the axle along +y. -->
-          <origin xyz="0 0 0" rpy="0 0 0"/>
-          <geometry><mesh filename="${loader_mesh_dir}/wheel.STL"/></geometry>
+          <origin xyz="0 0 0" rpy="${flip} 0 0"/>
+          <geometry><mesh filename="${loader_mesh_dir}/visual/wheel_tire.STL"/></geometry>
         </xacro:if>
-        <xacro:unless value="'$(arg mesh_visuals)' == 'true'">
+        <xacro:unless value="$(arg mesh_visuals)">
           <origin xyz="0 0 0" rpy="${pi / 2.0} 0 0"/>
           <geometry><cylinder radius="${nominal_wheel_radius}" length="${nominal_wheel_width}"/></geometry>
@@ -88,4 +96,11 @@
         <material name="loader_dark"/>
       </visual>
+      <xacro:if value="$(arg mesh_visuals)">
+        <visual>
+          <origin xyz="0 0 0" rpy="${flip} 0 0"/>
+          <geometry><mesh filename="${loader_mesh_dir}/visual/wheel_rim.STL"/></geometry>
+          <material name="wheel_rim"/>
+        </visual>
+      </xacro:if>
       <collision>
         <origin xyz="0 0 0" rpy="${pi / 2.0} 0 0"/>
@@ -98,5 +113,5 @@
     name="rear_frame" mass="7200" size_x="2.8" size_y="2.2" size_z="0.8"
     geometry_xyz="-1.4 0 0.15" material="loader_yellow"
-    mesh="${loader_mesh_dir}/rear_body.STL"/>
+    mesh="${loader_mesh_dir}/visual/rear_body.STL" glass="${True}"/>
   <joint name="base_to_rear_frame" type="fixed">
     <parent link="base_link"/>
@@ -107,5 +122,5 @@
     name="front_frame" mass="6200" size_x="3.0" size_y="2.2" size_z="0.75"
     geometry_xyz="1.5 0 0.15" material="loader_yellow"
-    mesh="${loader_mesh_dir}/front_body.STL"/>
+    mesh="${loader_mesh_dir}/visual/front_body.STL"/>
   <joint name="articulation_joint" type="revolute">
     <parent link="rear_frame"/>
@@ -127,5 +142,5 @@
     <dynamics damping="8000" friction="2000"/>
   </joint>
-  <xacro:wheel_link name="rear_left_wheel" mass="650"/>
+  <xacro:wheel_link name="rear_left_wheel" mass="650" flip="${pi}"/>
   <joint name="rear_left_wheel_joint" type="continuous">
     <parent link="rear_axle"/><child link="rear_left_wheel"/>
@@ -139,5 +154,5 @@
     <axis xyz="0 1 0"/><dynamics damping="50" friction="10"/>
   </joint>
-  <xacro:wheel_link name="front_left_wheel" mass="650"/>
+  <xacro:wheel_link name="front_left_wheel" mass="650" flip="${pi}"/>
   <joint name="front_left_wheel_joint" type="continuous">
     <parent link="front_frame"/><child link="front_left_wheel"/>
@@ -174,4 +189,8 @@
   </joint>
   <link name="lidar_link">
+    <visual>
+      <geometry><cylinder radius="0.10" length="0.16"/></geometry>
+      <material name="loader_dark"/>
+    </visual>
     <inertial>
       <mass value="2.0"/>
@@ -181,5 +200,6 @@
   <joint name="lidar_mount_joint" type="fixed">
     <parent link="rear_frame"/><child link="lidar_link"/>
-    <origin xyz="${-0.85 + lidar_off_xyz[0]} ${lidar_off_xyz[1]} ${2.25 + lidar_off_xyz[2]}"
+    <!-- Clear the L580 roof (maximum z=2.674 m in rear_frame). -->
+    <origin xyz="${-0.85 + lidar_off_xyz[0]} ${lidar_off_xyz[1]} ${2.85 + lidar_off_xyz[2]}"
       rpy="${lidar_off_rpy[0]} ${lidar_off_rpy[1]} ${lidar_off_rpy[2]}"/>
   </joint>
